File: poe-nrf-sentry.kicad_pcb (KiCad board)
At the start: 4 copper layers, 107 x 73 mm, 207 parts, among them J1 RJ45, J2 RJ45, J3 TAG-CONN, J4 Conn_02x20_Odd_Even, J5 USB-C, J6 MM8130-2600RA2, J7 DSUB DB9 MALE, Q1 NPN 40V 0.2A, Q2 N-CH 25V 0.22A, Q3 N-CH 100V 30A, Q4 N-CH 100V 30A, Q5 N-CH 100V 30A, Q6 N-CH 100V 30A, Q7 P-CH 30V 6A, SW1 SW_KMR211NGLFS_SMD, T1 S558-5999-U7-F, U1 NRF52840-QIAA-R, U15 BME688, U2 W5500, U3 KSZ8895RQXI-TR, U4 Si3474B-A01-IMR, U5 12A, U6 RS232_16-TSSOP_MAX3232IPWR, X1 MU00525-32.768K, Y1 XRCGB32M000F2P01R0, Y2 XRCGB25M000FAM10R0, Y3 XRCGB25M000FAM10R0

Commit message: latestL
Parts:
- added C82: 220uF 35V, Capacitor_SMD:CP_Elec_8x10.5, F.Cu at (82.8, 112.4)
- added C83: 220uF 35V, Capacitor_SMD:CP_Elec_8x10.5, F.Cu at (82.8, 121.4)
- added C84: 100nF 50V X7R, andium-capacitors:C_0402_1005Metric, B.Cu at (75.7, 120.0)
- added C85: 22uF 16V X5R, antmicro-footprints:C_0603_1608Metric, F.Cu at (72.9, 141.5)
- added C86: 22uF 16V X5R, antmicro-footprints:C_0603_1608Metric, F.Cu at (72.9, 142.8)
- added C87: 100nF 50V X7R, andium-capacitors:C_0402_1005Metric, B.Cu at (70.1, 135.2)
- added C88: 22uF 100V, Capacitor_SMD:CP_Elec_8x10.5, F.Cu at (82.7, 92.8)
- added C89: 22uF 100V, Capacitor_SMD:CP_Elec_8x10.5, F.Cu at (82.7, 101.8)
- added C90: 100nF 100V X7R, andium-capacitors:C_0603_1608Metric, B.Cu at (76.8, 97.0)
- added C91: 100nF 50V X7R, andium-capacitors:C_0402_1005Metric, B.Cu at (75.7, 114.8)
- moved +3V3D1 193.9 mm to (115.7, 160.9)
- moved GND2 193.9 mm to (115.7, 163.9)
- moved GND3 193.9 mm to (116.0, 169.2)
- moved POEAUTO1 193.9 mm to (110.7, 160.9)
- moved POEINT1 193.9 mm to (110.7, 163.9)
- moved POEOSS1 193.9 mm to (110.7, 167.0)
- moved POERST1 193.9 mm to (110.7, 170.1)
- moved POERST2 193.9 mm to (110.7, 173.1)
- moved PSCK1 193.9 mm to (118.8, 160.9)
- moved PSCS1 193.9 mm to (118.8, 163.9)
- moved PSDI1 193.9 mm to (121.8, 160.9)
- moved PSDO1 193.9 mm to (121.8, 163.9)
- moved VUSB1 193.9 mm to (116.0, 172.8)
- moved 3V3_LED1 36.0 mm to (65.2, 157.7)
- moved D9 36.0 mm to (82.7, 163.4)
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Routing:
- net PGND: track 44.0 -> 75.2 mm, vias 44 -> 65
- net /eth-port2/POE_BM: track 132.0 -> 105.7 mm, vias 10 -> 11
- net /poe-controller/G2: track 13.8 -> 39.1 mm
- net /poe-controller/G1: track 19.4 -> 44.8 mm
- net /poe-controller/S2: track 13.4 -> 38.8 mm
- net /poe-controller/S1: track 15.0 -> 40.3 mm
- net /poe-controller/S3: track 14.3 -> 30.9 mm, vias 2 -> 4
- net /poe-controller/G3: track 15.2 -> 30.7 mm
- net /eth-port2/POE_AM: track 108.2 -> 99.6 mm, vias 10 -> 12
- net GND: track 148.3 -> 156.4 mm, vias 210 -> 262
- net /poe-controller/S4: track 23.6 -> 16.0 mm, vias 2 -> 0
- net /nrf52840/RS232_MCU_RX: track 34.0 -> 27.5 mm
- net /nrf52840/RS232_MCU_DTR: track 33.7 -> 27.5 mm
- net /eth-sw/MOSI: track 20.4 -> 14.2 mm
- net /nrf52840/RS232_MCU_TX: track 33.5 -> 27.5 mm
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- added copper zone on In2.Cu, net +VPOE
- removed copper zone on In1.Cu, net GND
Other:
- outline, holes or cut-outs redrawn
